Commit message: couldnt figure out hownto do the xarco

File: milestone5_ws/src/robots_viz/urdf/robots_viz.urdf.xacro (robot description, xacro)
@@ -4,15 +4,15 @@
   <xacro:property name="L1" value="0.20" />
   <xacro:property name="L1radius" value="0.05" />
-  <xacro:property name="L2" value="0.15" />
-  <xacro:property name="L2radius" value="0.03" />
-  <xacro:property name="L3" value="0.08" />
-  <xacro:property name="L3radius" value="0.02" />
+  <xacro:property name="L2" value="0.08" />
+  <xacro:property name="L2radius" value="0.05" />
+  <xacro:property name="L3" value="0.06" />
+  <xacro:property name="L3radius" value="0.03" />
   <xacro:property name="eesize" value="0.05" />
-  <xacro:property name="J1MIN" value="${-pi/2}" />
-  <xacro:property name="J1MAX" value="${pi/2}" />
-  <xacro:property name="J2MIN" value="-0.08" />
-  <xacro:property name="J2MAX" value="0.08" />
-  <xacro:property name="J3MIN" value="${-pi}" />
-  <xacro:property name="J3MAX" value="${pi}" />
+  <xacro:property name="J1MIN" value="0" />
+  <xacro:property name="J1MAX" value="0.20" />
+  <xacro:property name="J2MIN" value="${-pi/2}" />
+  <xacro:property name="J2MAX" value="${pi/2}" />
+  <xacro:property name="J3MIN" value="${0}" />
+  <xacro:property name="J3MAX" value="${0.06}" />
   <material name="blue">
     <color rgba="0.2 0.4 0.65 1" />
@@ -27,5 +27,6 @@
       <origin xyz="0 0 ${-L1/2}" />
       <geometry>
-        <cylinder radius="${L1radius}" length="${L1}" />
+        <box size="${L1radius} ${L1radius} ${L1}" />
+        <!-- <cylinder radius="${L1radius}" length="${L1}" /> -->
       </geometry>
       <material name="blue" />
@@ -34,7 +35,7 @@
   <link name="link2">
     <visual name="link2">
-      <origin xyz="0 0 0" />
+      <origin xyz="0 0 ${-L2}" />
       <geometry>
-        <cylinder radius="${L2radius}" length="${2*L2}" />
+         <box size="${L2radius} ${L2radius} ${L2}"/>
       </geometry>
       <material name="blue" />
@@ -43,5 +44,5 @@
   <link name="link3">
     <visual name="link3">
-      <origin xyz="0 0 ${L3/2}" />
+      <origin xyz="0 0 0" />
       <geometry>
         <cylinder radius="${L3radius}" length="${L3}" />
@@ -64,29 +65,29 @@
     <origin xyz="${-(L2+L3)} 0 0" rpy="0 0 ${pi/2}" />
   </joint>
-  <joint name="joint1" type="revolute">
+  <joint name="base_to_l1" type="fixed">
     <parent link="base" />
     <child link="link1" />
-    <origin xyz="0 0 ${L1}" rpy="0 0 0" />
-    <axis xyz="0 0 1" />
+    <origin xyz="0 0 ${L1}" rpy="0 0 ${-pi/2}" />
+  </joint>
+  <joint name="joint1" type="prismatic">
+    <parent link="link1" />
+    <child link="link2" />
+    <origin xyz="0 0 0" rpy="0 ${-pi/2} 0" />
+    <axis xyz="1 0 0" />
     <limit lower="${J1MIN}" upper="${J1MAX}" effort="1" velocity="1" />
   </joint>
-  <joint name="joint2" type="prismatic">
-    <parent link="link1" />
-    <child link="link2" />
-    <origin xyz="0 0 0" rpy="${pi/2} 0 0" />
-    <axis xyz="0 0 1" />
+  <joint name="joint2" type="revolute">
+    <parent link="link2" />
+    <child link="link3" />
+    <origin xyz="0 0 0" rpy="0 0 0" />
+    <axis xyz="1 0 0" />
     <limit lower="${J2MIN}" upper="${J2MAX}" effort="1" velocity="1" />
   </joint>
-  <joint name="joint3" type="revolute">
-    <parent link="link2" />
-    <child link="link3" />
-    <origin xyz="0 0 ${L2}" rpy="0 0 0" />
-    <axis xyz="0 0 1" />
-    <limit lower="${J3MIN}" upper="${J3MAX}" effort="1" velocity="1" />
-  </joint>
-  <joint name="ee_in_link3" type="fixed">
+  <joint name="ee_in_link3" type="prismatic">
     <parent link="link3" />
     <child link="ee" />
-    <origin xyz="0 0 ${L3}" rpy="0 0 0" />
+    <origin xyz="0 0 ${-(L2+L3)}" rpy="0 ${pi}  0" />
+    <limit lower="${J3MIN}" upper="${J3MAX}" effort="1" velocity="1" />
+    <axis xyz="0 0 1" />
   </joint>
 </robot>

Commit message: might have  it wright

File: milestone5_ws/src/robots_viz/urdf/robots_viz.urdf.xacro (robot description, xacro)
@@ -9,10 +9,10 @@
   <xacro:property name="L3radius" value="0.03" />
   <xacro:property name="eesize" value="0.05" />
-  <xacro:property name="J1MIN" value="0" />
-  <xacro:property name="J1MAX" value="0.20" />
+  <xacro:property name="J1MIN" value="-0.08" />
+  <xacro:property name="J1MAX" value="0.08" />
   <xacro:property name="J2MIN" value="${-pi/2}" />
   <xacro:property name="J2MAX" value="${pi/2}" />
-  <xacro:property name="J3MIN" value="${0}" />
-  <xacro:property name="J3MAX" value="${0.06}" />
+  <xacro:property name="J3MIN" value="${-0.04}" />
+  <xacro:property name="J3MAX" value="${0.04}" />
   <material name="blue">
     <color rgba="0.2 0.4 0.65 1" />
@@ -25,5 +25,5 @@
   <link name="link1">
     <visual name="link1">
-      <origin xyz="0 0 ${-L1/2}" />
+      <origin xyz="0 0 ${L1/2}" />
       <geometry>
         <box size="${L1radius} ${L1radius} ${L1}" />
@@ -35,5 +35,5 @@
   <link name="link2">
     <visual name="link2">
-      <origin xyz="0 0 ${-L2}" />
+      <origin xyz="0 0 ${-L2/2}" />
       <geometry>
          <box size="${L2radius} ${L2radius} ${L2}"/>
@@ -68,10 +68,10 @@
     <parent link="base" />
     <child link="link1" />
-    <origin xyz="0 0 ${L1}" rpy="0 0 ${-pi/2}" />
+    <origin xyz="0 0 0" rpy="0 0 ${-pi/2}" />
   </joint>
   <joint name="joint1" type="prismatic">
     <parent link="link1" />
     <child link="link2" />
-    <origin xyz="0 0 0" rpy="0 ${-pi/2} 0" />
+    <origin xyz="0 0 ${L1}" rpy="0 ${-pi/2} 0" />
     <axis xyz="1 0 0" />
     <limit lower="${J1MIN}" upper="${J1MAX}" effort="1" velocity="1" />
@@ -80,5 +80,5 @@
     <parent link="link2" />
     <child link="link3" />
-    <origin xyz="0 0 0" rpy="0 0 0" />
+    <origin xyz="0 0 ${-L2}" rpy="${-pi/2} 0 0" />
     <axis xyz="1 0 0" />
     <limit lower="${J2MIN}" upper="${J2MAX}" effort="1" velocity="1" />
@@ -87,7 +87,7 @@
     <parent link="link3" />
     <child link="ee" />
-    <origin xyz="0 0 ${-(L2+L3)}" rpy="0 ${pi}  0" />
+    <origin xyz="0 0 0" rpy="0 0  0" />
     <limit lower="${J3MIN}" upper="${J3MAX}" effort="1" velocity="1" />
-    <axis xyz="0 0 1" />
+    <axis xyz="0 1 0" />
   </joint>
 </robot>

Commit message: pretty sure finished dh notaiton for robot

File: milestone5_ws/src/robots_viz/urdf/robots_viz.urdf.xacro (robot description, xacro)
@@ -2,16 +2,10 @@
 <!DOCTYPE xml>
 <robot xmlns:xacro="http://www.ros.org/wiki/xacro" name="robots_viz">
-  <xacro:property name="L0" value="0.056" />
-  <xacro:property name="L0radius" value="0.03" />
-  <xacro:property name="L1" value="0.082" />
-  <xacro:property name="L1radius" value="0.02" />
-  <xacro:property name="L2" value="0.145" />
+  <xacro:property name="L1" value="0.20" />
+  <xacro:property name="L1radius" value="0.05" />
+  <xacro:property name="L2" value="0.08" />
   <xacro:property name="L2radius" value="0.05" />
-  <xacro:property name="L3" value="0.147" />
+  <xacro:property name="L3" value="0.06" />
   <xacro:property name="L3radius" value="0.03" />
-  <xacro:property name="L4" value="0.06" />
-  <xacro:property name="L4radius" value="0.03" />
-  <xacro:property name="L5" value="0.07" />
-  <xacro:property name="L5radius" value="0.03" />
   <xacro:property name="eesize" value="0.05" />
   <xacro:property name="J1MIN" value="-0.08" />
@@ -19,6 +13,6 @@
   <xacro:property name="J2MIN" value="${-pi/2}" />
   <xacro:property name="J2MAX" value="${pi/2}" />
-  <xacro:property name="J3MIN" value="${-0.04}" />
-  <xacro:property name="J3MAX" value="${0.04}" />
+  <xacro:property name="J3MIN" value="${0}" />
+  <xacro:property name="J3MAX" value="${0.06}" />
   <material name="blue">
     <color rgba="0.2 0.4 0.65 1" />
@@ -29,9 +23,9 @@
   <link name="world" />
   <link name="base" />
-  <link name="link0">
-    <visual name="link0">
-      <origin xyz="0 0 ${L0/2}" />
+  <link name="link1">
+    <visual name="link1">
+      <origin xyz="0 0 ${-L1/2}" />
       <geometry>
-        <box size="${L0radius} ${L0radius} ${L0}" />
+        <box size="${L1radius} ${L1radius} ${L1 + 0.1}" />
         <!-- <cylinder radius="${L1radius}" length="${L1}" /> -->
       </geometry>
@@ -39,19 +33,9 @@
     </visual>
   </link>
-  <link name="link1">
-    <visual name="link1">
-      <origin xyz="0 0 ${L1/2}" />
+  <link name="link2">
+    <visual name="link2">
+      <origin xyz="0 ${L2/2} 0"  rpy="0 0 0"/>
       <geometry>
-        <box size="${L1radius} ${L1radius} ${L1}" />
-        <!-- <cylinder radius="${L1radius}" length="${L1}" /> -->
-      </geometry>
-      <material name="blue" />
-    </visual>
-  </link>
-  <!-- <link name="link2">
-    <visual name="link2">
-      <origin xyz="0 0 ${L2/2}" rpy = "0 0 0"/>
-      <geometry>
-         <box size="${L2radius} ${L2radius} ${L2}"/>
+         <box size="${L2radius} ${L2} ${L2radius} "/>
       </geometry>
       <material name="blue" />
@@ -60,5 +44,5 @@
   <link name="link3">
     <visual name="link3">
-      <origin xyz="0 0 0" rpy = "0 ${pi/2} 0"/>
+      <origin xyz="0 0 0" />
       <geometry>
         <cylinder radius="${L3radius}" length="${L3}" />
@@ -67,25 +51,7 @@
     </visual>
   </link>
-   <link name="link4">
-    <visual name="link4">
-      <origin xyz="0 0 0" rpy = "0 ${pi/2} 0"/>
-      <geometry>
-        <cylinder radius="${L4radius}" length="${L4}" />
-      </geometry>
-      <material name="blue" />
-    </visual>
-  </link>
-    <link name="link5">
-    <visual name="link5">
-      <origin xyz="0 0 0" rpy = "0 ${pi/2} 0"/>
-      <geometry>
-        <cylinder radius="${L5radius}" length="${L5}" />
-      </geometry>
-      <material name="blue" />
-    </visual>
-  </link>
   <link name="ee">
     <visual name="ee">
-      <origin xyz="0 0 0" />
+      <origin xyz="0 0 0.06" />
       <geometry>
         <box size="${eesize} ${eesize} ${eesize}" />
@@ -93,26 +59,33 @@
       <material name="yellow" />
     </visual>
-  </link> -->
+    <visual name="eeArm">
+      <origin xyz="0 0 0" />
+      <geometry>
+        <box size="${eesize/2} ${eesize/2} 0.1" />
+      </geometry>
+      <material name="blue" />
+    </visual>
+  </link>
   <joint name="base_in_world" type="fixed">
     <parent link="world" />
     <child link="base" />
-    <origin xyz="${-(L3+L3)} 0 0" rpy="0 0 ${pi/2}" />
+    <origin xyz="${-(L2+L3)} 0 0" rpy="0 0 ${pi/2}" />
   </joint>
-  <joint name="joint0" type="fixed">
+  <joint name="base_to_l1" type="fixed">
     <parent link="base" />
-    <child link="link0" />
+    <child link="link1" />
     <origin xyz="0 0 ${L1}" rpy="0 0 ${-pi/2}" />
   </joint>
-  <joint name="joint1" type="revolute">
-    <parent link="link0" />
-    <child link="link1" />
-    <origin xyz="0 0 0" rpy="0 0 0" />
+  <joint name="joint1" type="prismatic">
+    <parent link="link1" />
+    <child link="link2" />
+    <origin xyz="0 0 0" rpy="0 0 ${-pi/2}" />
     <axis xyz="0 0 1" />
     <limit lower="${J1MIN}" upper="${J1MAX}" effort="1" velocity="1" />
   </joint>
-  <!-- <joint name="joint2" type="revolute">
+  <joint name="joint2" type="revolute">
     <parent link="link2" />
     <child link="link3" />
-    <origin xyz="0 0 0" rpy="0 0 0" />
+    <origin xyz="0 ${L2} 0" rpy="0 0 0" />
     <axis xyz="0 0 1" />
     <limit lower="${J2MIN}" upper="${J2MAX}" effort="1" velocity="1" />
@@ -121,7 +94,7 @@
     <parent link="link3" />
     <child link="ee" />
-    <origin xyz="0 0 0" rpy="0 0  0" />
+    <origin xyz="0 0 0" rpy=" ${-pi/2} 0 0 " />
     <limit lower="${J3MIN}" upper="${J3MAX}" effort="1" velocity="1" />
     <axis xyz="0 0 1" />
-  </joint> -->
+  </joint>
 </robot>

Commit message: finsihed milestone 5 and finsihed 6.1, 6.2, 6.3 on 6.4

File: milestone5_ws/src/robots_viz/urdf/robots_viz.urdf.xacro (robot description, xacro)
@@ -13,6 +13,6 @@
   <xacro:property name="J2MIN" value="${-pi/2}" />
   <xacro:property name="J2MAX" value="${pi/2}" />
-  <xacro:property name="J3MIN" value="${0}" />
-  <xacro:property name="J3MAX" value="${0.06}" />
+  <xacro:property name="J3MIN" value="${-0.04}" />
+  <xacro:property name="J3MAX" value="${0.04}" />
   <material name="blue">
     <color rgba="0.2 0.4 0.65 1" />
