Commit message: finished most of the milestone just need to do indiviuvutal and 5.5

File: dobot_ws/src/dobot_twin_viz/urdf/dobot_twin_viz.urdf.xacro (robot description, xacro)
@@ -1,7 +1,7 @@
 <?xml version="1.0" encoding="UTF-8"?>
 <!DOCTYPE xml>
-<robot xmlns:xacro="http://www.ros.org/wiki/xacro" name="robots_viz">
+<robot xmlns:xacro="http://www.ros.org/wiki/xacro" name="dobot_twin_viz">
   <xacro:property name="L0" value="0.056" />
-  <xacro:property name="L0radius" value="0.03" />
+  <xacro:property name="L0radius" value="0.1" />
   <xacro:property name="L1" value="0.082" />
   <xacro:property name="L1radius" value="0.02" />
@@ -15,10 +15,12 @@
   <xacro:property name="L5radius" value="0.03" />
   <xacro:property name="eesize" value="0.05" />
-  <xacro:property name="J1MIN" value="0" />
-  <xacro:property name="J1MAX" value="0.20" />
-  <xacro:property name="J2MIN" value="${-pi/2}" />
-  <xacro:property name="J2MAX" value="${pi/2}" />
-  <xacro:property name="J3MIN" value="${0}" />
-  <xacro:property name="J3MAX" value="${0.06}" />
+  <xacro:property name="J1MIN" value="${-pi/2}" />
+  <xacro:property name="J1MAX" value="${pi/2}" />
+  <xacro:property name="J2MIN" value="0" />
+  <xacro:property name="J2MAX" value="${70*pi/180}" />
+  <xacro:property name="J3MIN" value="${15*pi/180}" />
+  <xacro:property name="J3MAX" value="${40*pi/180}" />
+  <xacro:property name="J4MIN" value="${-90*pi/180}" />
+  <xacro:property name="J4MAX" value="${90*pi/180}" />
   <material name="blue">
     <color rgba="0.2 0.4 0.65 1" />
@@ -49,5 +51,5 @@
     </visual>
   </link>
-  <!-- <link name="link2">
+ <link name="link2">
     <visual name="link2">
       <origin xyz="0 0 ${L2/2}" rpy = "0 0 0"/>
@@ -58,7 +60,7 @@
     </visual>
   </link>
-  <link name="link3">
+    <link name="link3">
     <visual name="link3">
-      <origin xyz="0 0 0" rpy = "0 ${pi/2} 0"/>
+      <origin xyz="${L3/2}  0 0" rpy = "0 ${pi/2} 0"/>
       <geometry>
         <cylinder radius="${L3radius}" length="${L3}" />
@@ -67,9 +69,20 @@
     </visual>
   </link>
-   <link name="link4">
+  <link name="link4">
     <visual name="link4">
-      <origin xyz="0 0 0" rpy = "0 ${pi/2} 0"/>
+      <origin xyz="${L4/2} 0 0" rpy = "0 ${pi/2} 0"/>
       <geometry>
-        <cylinder radius="${L4radius}" length="${L4}" />
+        <!-- <cylinder radius="${L3radius}" length="${L3}" /> -->
+        <box size="${L4radius} ${L4radius} ${L4}" />
+      </geometry>
+      <material name="blue" />
+    </visual>
+  </link>
+  <link name="link4_mimic">
+    <visual name="link4_mimic">
+      <origin xyz="0 0 0" rpy = "0 0 0"/>
+      <geometry>
+        <!-- <cylinder radius="${L3radius}" length="${L3}" /> -->
+        <box size="0 0 0" />
       </geometry>
       <material name="blue" />
@@ -78,5 +91,5 @@
     <link name="link5">
     <visual name="link5">
-      <origin xyz="0 0 0" rpy = "0 ${pi/2} 0"/>
+      <origin xyz="0 0 ${-L5/2}" rpy = "0 0 0"/>
       <geometry>
         <cylinder radius="${L5radius}" length="${L5}" />
@@ -85,4 +98,5 @@
     </visual>
   </link>
+<!--
   <link name="ee">
     <visual name="ee">
@@ -102,14 +116,51 @@
     <parent link="base" />
     <child link="link0" />
-    <origin xyz="0 0 ${L1}" rpy="0 0 ${-pi/2}" />
+    <origin xyz="0 0 0" rpy="0 0 ${-pi/2}" />
   </joint>
-  <joint name="joint1" type="revolute">
+  <joint name="J1" type="revolute">
     <parent link="link0" />
     <child link="link1" />
-    <origin xyz="0 0 0" rpy="0 0 0" />
+    <origin xyz="0 0 ${L0}" rpy="0 ${-pi} 0" />
     <axis xyz="0 0 1" />
     <limit lower="${J1MIN}" upper="${J1MAX}" effort="1" velocity="1" />
   </joint>
-  <!-- <joint name="joint2" type="revolute">
+  <joint name="J2" type="revolute">
+    <parent link="link1" />
+    <child link="link2" />
+    <origin xyz="0 0 ${-L1}" rpy="0 ${-pi} 0" />
+    <axis xyz="0 1 0" />
+    <limit lower="${J2MIN}" upper="${J2MAX}" effort="1" velocity="1" />
+  </joint>
+  <joint name="J3" type="revolute">
+    <parent link="link2" />
+    <child link="link3" />
+    <origin xyz="0 0 ${L2}" rpy="0 0 0" />
+    <axis xyz="0 1 0" />
+    <limit lower="${J3MIN}" upper="${J3MAX}" effort="1" velocity="1" />
+  </joint>
+  <joint name="joint4_1" type="revolute">
+    <parent link="link3" />
+    <child link="link4_mimic" />
+    <origin xyz="${L3} 0 0" rpy="0 0 0" />
+    <axis xyz="0 1 0" />
+    <limit lower="${J1MIN}" upper="${J1MAX}" effort="1" velocity="1" />
+    <mimic joint = "J3" multiplier="-1" offset = "0"/>
+  </joint>
+  <joint name="joint4_2" type="revolute">
+    <parent link="link4_mimic" />
+    <child link="link4" />
+    <origin xyz="0   0 0" rpy="0 0 0" />
+    <axis xyz="0 1 0" />
+    <limit lower="${J1MIN}" upper="${J1MAX}" effort="1" velocity="1" />
+    <mimic joint = "J2" multiplier="-1" offset = "0"/>
+  </joint>
+      <joint name="J4" type="revolute">
+    <parent link="link4" />
+    <child link="link5" />
+    <origin xyz="${L4} 0 0" rpy="0 0 ${-pi}" />
+    <axis xyz="0 0 1" />
+    <limit lower="${J4MIN}" upper="${J4MAX}" effort="1" velocity="1" />
+  </joint>
+  <!-- <joint name="J2" type="revolute">
     <parent link="link2" />
     <child link="link3" />

File: dobot_ws/src/dobot_viz/urdf/dobot_viz.urdf.xacro (robot description, xacro)
@@ -1,7 +1,7 @@
 <?xml version="1.0" encoding="UTF-8"?>
 <!DOCTYPE xml>
-<robot xmlns:xacro="http://www.ros.org/wiki/xacro" name="robots_viz">
+<robot xmlns:xacro="http://www.ros.org/wiki/xacro" name="dobot_viz">
   <xacro:property name="L0" value="0.056" />
-  <xacro:property name="L0radius" value="0.03" />
+  <xacro:property name="L0radius" value="0.1" />
   <xacro:property name="L1" value="0.082" />
   <xacro:property name="L1radius" value="0.02" />
@@ -15,10 +15,20 @@
   <xacro:property name="L5radius" value="0.03" />
   <xacro:property name="eesize" value="0.05" />
-  <xacro:property name="J1MIN" value="0" />
-  <xacro:property name="J1MAX" value="0.20" />
-  <xacro:property name="J2MIN" value="${-pi/2}" />
-  <xacro:property name="J2MAX" value="${pi/2}" />
-  <xacro:property name="J3MIN" value="${0}" />
-  <xacro:property name="J3MAX" value="${0.06}" />
+  J1MIN = -90
+J1MAX = 90
+J2MIN = 0
+J2MAX = 70
+J3MIN = -15
+J3MAX = 40
+J4MIN = -90
+J4MAX = 90
+  <xacro:property name="J1MIN" value="${-pi/2}" />
+  <xacro:property name="J1MAX" value="${pi/2}" />
+  <xacro:property name="J2MIN" value="0" />
+  <xacro:property name="J2MAX" value="${70*pi/180}" />
+  <xacro:property name="J3MIN" value="${15*pi/180}" />
+  <xacro:property name="J3MAX" value="${40*pi/180}" />
+  <xacro:property name="J4MIN" value="${-90*pi/180}" />
+  <xacro:property name="J4MAX" value="${90*pi/180}" />
   <material name="blue">
     <color rgba="0.2 0.4 0.65 1" />
@@ -49,5 +59,5 @@
     </visual>
   </link>
-  <!-- <link name="link2">
+ <link name="link2">
     <visual name="link2">
       <origin xyz="0 0 ${L2/2}" rpy = "0 0 0"/>
@@ -58,7 +68,7 @@
     </visual>
   </link>
-  <link name="link3">
+    <link name="link3">
     <visual name="link3">
-      <origin xyz="0 0 0" rpy = "0 ${pi/2} 0"/>
+      <origin xyz="${L3/2}  0 0" rpy = "0 ${pi/2} 0"/>
       <geometry>
         <cylinder radius="${L3radius}" length="${L3}" />
@@ -67,9 +77,20 @@
     </visual>
   </link>
-   <link name="link4">
+  <link name="link4">
     <visual name="link4">
-      <origin xyz="0 0 0" rpy = "0 ${pi/2} 0"/>
+      <origin xyz="${L4/2} 0 0" rpy = "0 ${pi/2} 0"/>
       <geometry>
-        <cylinder radius="${L4radius}" length="${L4}" />
+        <!-- <cylinder radius="${L3radius}" length="${L3}" /> -->
+        <box size="${L4radius} ${L4radius} ${L4}" />
+      </geometry>
+      <material name="blue" />
+    </visual>
+  </link>
+  <link name="link4_mimic">
+    <visual name="link4_mimic">
+      <origin xyz="0 0 0" rpy = "0 0 0"/>
+      <geometry>
+        <!-- <cylinder radius="${L3radius}" length="${L3}" /> -->
+        <box size="0 0 0" />
       </geometry>
       <material name="blue" />
@@ -78,5 +99,5 @@
     <link name="link5">
     <visual name="link5">
-      <origin xyz="0 0 0" rpy = "0 ${pi/2} 0"/>
+      <origin xyz="0 0 ${-L5/2}" rpy = "0 0 0"/>
       <geometry>
         <cylinder radius="${L5radius}" length="${L5}" />
@@ -85,4 +106,5 @@
     </visual>
   </link>
+<!--
   <link name="ee">
     <visual name="ee">
@@ -102,12 +124,49 @@
     <parent link="base" />
     <child link="link0" />
-    <origin xyz="0 0 ${L1}" rpy="0 0 ${-pi/2}" />
+    <origin xyz="0 0 0" rpy="0 0 ${-pi/2}" />
   </joint>
   <joint name="joint1" type="revolute">
     <parent link="link0" />
     <child link="link1" />
-    <origin xyz="0 0 0" rpy="0 0 0" />
+    <origin xyz="0 0 ${L0}" rpy="0 ${-pi} 0" />
     <axis xyz="0 0 1" />
     <limit lower="${J1MIN}" upper="${J1MAX}" effort="1" velocity="1" />
+  </joint>
+  <joint name="joint2" type="revolute">
+    <parent link="link1" />
+    <child link="link2" />
+    <origin xyz="0 0 ${-L1}" rpy="0 ${-pi} 0" />
+    <axis xyz="0 1 0" />
+    <limit lower="${J2MIN}" upper="${J2MAX}" effort="1" velocity="1" />
+  </joint>
+  <joint name="joint3" type="revolute">
+    <parent link="link2" />
+    <child link="link3" />
+    <origin xyz="0 0 ${L2}" rpy="0 0 0" />
+    <axis xyz="0 1 0" />
+    <limit lower="${J3MIN}" upper="${J3MAX}" effort="1" velocity="1" />
+  </joint>
+  <joint name="joint4_1" type="revolute">
+    <parent link="link3" />
+    <child link="link4_mimic" />
+    <origin xyz="${L3} 0 0" rpy="0 0 0" />
+    <axis xyz="0 1 0" />
+    <limit lower="${J1MIN}" upper="${J1MAX}" effort="1" velocity="1" />
+    <mimic joint = "joint3" multiplier="-1" offset = "0"/>
+  </joint>
+  <joint name="joint4_2" type="revolute">
+    <parent link="link4_mimic" />
+    <child link="link4" />
+    <origin xyz="0   0 0" rpy="0 0 0" />
+    <axis xyz="0 1 0" />
+    <limit lower="${J1MIN}" upper="${J1MAX}" effort="1" velocity="1" />
+    <mimic joint = "joint2" multiplier="-1" offset = "0"/>
+  </joint>
+      <joint name="joint5" type="revolute">
+    <parent link="link4" />
+    <child link="link5" />
+    <origin xyz="${L4} 0 0" rpy="0 0 ${-pi}" />
+    <axis xyz="0 0 1" />
+    <limit lower="${J4MIN}" upper="${J4MAX}" effort="1" velocity="1" />
   </joint>
   <!-- <joint name="joint2" type="revolute">

Commit message: think i got a rvis wokring

File: dobot_ws/src/dobot_twin_viz/urdf/dobot_twin_viz.urdf.xacro (robot description, xacro)
@@ -13,6 +13,6 @@
   <xacro:property name="L4radius" value="0.03" />
   <xacro:property name="L5" value="0.07" />
-  <xacro:property name="L5radius" value="0.03" />
-  <xacro:property name="eesize" value="0.05" />
+  <xacro:property name="L5radius" value="0.01" />
+  <xacro:property name="eesize" value="0.025" />
   <xacro:property name="J1MIN" value="${-pi/2}" />
   <xacro:property name="J1MAX" value="${pi/2}" />
@@ -28,4 +28,7 @@
   <material name="yellow">
     <color rgba="1 0.85 0 1" />
+  </material>
+  <material name="green">
+    <color rgba="0 0.85 0 1" />
   </material>
   <link name="world" />
@@ -98,5 +101,4 @@
     </visual>
   </link>
-<!--
   <link name="ee">
     <visual name="ee">
@@ -107,9 +109,28 @@
       <material name="yellow" />
     </visual>
-  </link> -->
+  </link>
+  <link name="end_block">
+    <visual name="end_block">
+      <origin xyz="0 0 0" />
+      <geometry>
+        <box size="${eesize} ${eesize} ${eesize}" />
+      </geometry>
+      <material name="green" />
+    </visual>
+  </link>
   <joint name="base_in_world" type="fixed">
     <parent link="world" />
     <child link="base" />
     <origin xyz="${-(L3+L3)} 0 0" rpy="0 0 ${pi/2}" />
+  </joint>
+    <joint name="first_box" type="fixed">
+    <parent link="world" />
+    <child link="ee" />
+    <origin xyz="0.092 -0.201 0" rpy="0 0 ${pi/2}" />
+  </joint>
+<joint name="last_box" type="fixed">
+    <parent link="world" />
+    <child link="end_block" />
+    <origin xyz="0.09 0.226 ${eesize*3 }" rpy="0 0 ${pi/2}" />
   </joint>
   <joint name="joint0" type="fixed">
